Commit message: adding links to 1 large urdf for now

File: v2mini_description/urdf/v2mini_base.urdf.xacro (robot description, xacro)
@@ -9,11 +9,28 @@
   <xacro:property name="wheel_radius" value="0.03" />
   <xacro:property name="wheel_offset_radial" value="0.15" />
+  <!-- torso properties -->
+  <xacro:property name="torso_offset_z" value="0.175" />
+  <xacro:property name="torso_width" value="0.2373" />
+  <!-- head properties -->
+  <xacro:property name="head_offset_z" value="0.2" />
+  <!-- arm properties -->
+  <xacro:property name="motor_depth" value="0.04175" />
   <!-- materials -->
   <material name="white">
-    <color rgba="0.7 0.7 0.7 1"/>
+    <color rgba="0.6 0.6 0.6 1"/>
+  </material>
+  <material name="blue">
+    <color rgba="0.3 0.3 0.9 1"/>
   </material>
   <material name="black">
-    <color rgba="0 0 0 1"/>
+    <color rgba="0.1 0.1 0.1 1"/>
   </material>
+  <material name="grey">
+    <color rgba="0.4 0.4 0.4 1"/>
+  </material>
+  <material name="yellow">
+    <color rgba="0.5 0.5 0.1 1"/>
+  </material>
+  <!-- **** BASE **** -->
   <link name="base_link">
     <visual>
@@ -22,5 +39,5 @@
         <mesh filename="package://v2mini_description/meshes/base/base.stl" />
       </geometry>
-      <material name="white"/>
+      <material name="blue"/>
     </visual>
     <collision>
@@ -53,3 +70,110 @@
   <xacro:wheel prefix="left" reflect="1" rotate="1"/>
   <xacro:wheel prefix="right" reflect="-1" rotate="1"/>
+  <!-- **** TORSO **** -->
+  <link name="torso_link">
+    <visual>
+      <origin xyz="0 0 ${torso_offset_z}" rpy="0 0 0" />
+      <geometry>
+        <mesh filename="package://v2mini_description/meshes/torso/torso.stl" />
+      </geometry>
+      <material name="white"/>
+    </visual>
+  </link>
+  <joint name="torso_slide" type="prismatic">
+    <parent link="base_link"/>
+    <child link="torso_link"/>
+    <origin xyz="0 0 ${torso_offset_z}"/>
+    <axis xyz="0 0 1"/>
+    <limit effort="1000.0" lower="-0.04" upper="0.04" velocity="0.5"/>
+  </joint>
+  <!-- **** HEAD **** -->
+  <link name="head_link">
+    <visual>
+      <origin xyz="0 0 ${-head_offset_z*2-0.065}" rpy="0 0 0" />
+      <geometry>
+        <mesh filename="package://v2mini_description/meshes/head/head.stl" />
+      </geometry>
+      <material name="yellow"/>
+    </visual>
+  </link>
+  <joint name="head_joint" type="continuous">
+    <parent link="torso_link"/>
+    <child link="head_link"/>
+    <origin xyz="0 0 ${head_offset_z}"/>
+    <axis xyz="0 0 1"/>
+  </joint>
+  <!-- **** ARM **** -->
+  <link name="arm_link1">
+    <visual>
+      <origin xyz="${torso_width/2} 0 -0.41" rpy="0 0 0" />
+      <geometry>
+        <mesh filename="package://v2mini_description/meshes/arm/arm_link1.stl" />
+      </geometry>
+      <material name="grey"/>
+    </visual>
+  </link>
+  <joint name="arm_joint_1" type="fixed">
+    <parent link="torso_link"/>
+    <child link="arm_link1"/>
+    <origin xyz="${-torso_width/2} 0 0.164"/>
+  </joint>
+  <link name="arm_link2">
+    <visual>
+      <origin xyz="${torso_width/2+motor_depth} 0 -0.41" rpy="0 0 0" />
+      <geometry>
+        <mesh filename="package://v2mini_description/meshes/arm/arm_link2.stl" />
+      </geometry>
+      <material name="yellow"/>
+    </visual>
+  </link>
+  <joint name="arm_joint_2" type="continuous">
+    <parent link="arm_link1"/>
+    <child link="arm_link2"/>
+    <origin xyz="${-motor_depth} 0 0"/>
+  </joint>
+  <link name="arm_link3">
+    <visual>
+      <origin xyz="${torso_width/2+motor_depth+0.025} 0 -0.41" rpy="0 0 0" />
+      <geometry>
+        <mesh filename="package://v2mini_description/meshes/arm/arm_link3.stl" />
+      </geometry>
+      <material name="grey"/>
+    </visual>
+  </link>
+  <joint name="arm_joint_3" type="continuous">
+    <parent link="arm_link2"/>
+    <child link="arm_link3"/>
+    <axis xyz="0 1 0"/>
+    <origin xyz="-0.027 0 0"/>
+  </joint>
+  <link name="arm_link4">
+    <visual>
+      <origin xyz="${torso_width/2+motor_depth+0.1115} 0 -0.41" rpy="0 0 0" />
+      <geometry>
+        <mesh filename="package://v2mini_description/meshes/arm/arm_link4.stl" />
+      </geometry>
+      <material name="yellow"/>
+    </visual>
+  </link>
+  <joint name="arm_joint_4" type="continuous">
+    <parent link="arm_link3"/>
+    <child link="arm_link4"/>
+    <axis xyz="1 0 0"/>
+    <origin xyz="-0.0855 0 0"/>
+  </joint>
+  <link name="arm_link5">
+    <visual>
+      <origin xyz="0 0 -0.41" rpy="0 0 0" />
+      <geometry>
+        <mesh filename="package://v2mini_description/meshes/arm/arm_link5.stl" />
+      </geometry>
+      <material name="grey"/>
+    </visual>
+  </link>
+  <joint name="arm_joint_5" type="continuous">
+    <parent link="arm_link4"/>
+    <child link="arm_link5"/>
+    <axis xyz="0 0 1"/>
+    <origin xyz="0 0 0"/>
+  </joint>
 </robot>
