Commit message: moved materials back into individ urdfs

File: v2mini_description/urdf/v2mini_body.urdf.xacro (robot description, xacro)
@@ -1,4 +1,23 @@
 <?xml version="1.0"?>
 <robot xmlns:xacro="http://www.ros.org/wiki/xacro" name="v2mini">
+  <!-- materials -->
+  <material name="white">
+    <color rgba="0.6 0.6 0.6 1"/>
+  </material>
+  <material name="blue">
+    <color rgba="0.3 0.3 0.9 1"/>
+  </material>
+  <material name="black">
+    <color rgba="0.2 0.2 0.2 1"/>
+  </material>
+  <material name="grey">
+    <color rgba="0.4 0.4 0.4 1"/>
+  </material>
+  <material name="yellow">
+    <color rgba="0.5 0.5 0.1 1"/>
+  </material>
+  <material name="red">
+    <color rgba="0.6 0.2 0.2 1"/>
+  </material>
   <xacro:property name="pi" value="3.14159" />
   <!-- base properties -->

File: v2mini_description/urdf/v2mini_robot.urdf.xacro (robot description, xacro)
@@ -1,23 +1,4 @@
 <?xml version="1.0"?>
 <robot xmlns:xacro="http://www.ros.org/wiki/xacro" name="v2mini">
-  <!-- materials -->
-  <material name="white">
-    <color rgba="0.6 0.6 0.6 1"/>
-  </material>
-  <material name="blue">
-    <color rgba="0.3 0.3 0.9 1"/>
-  </material>
-  <material name="black">
-    <color rgba="0.2 0.2 0.2 1"/>
-  </material>
-  <material name="grey">
-    <color rgba="0.4 0.4 0.4 1"/>
-  </material>
-  <material name="yellow">
-    <color rgba="0.5 0.5 0.1 1"/>
-  </material>
-  <material name="red">
-    <color rgba="0.6 0.2 0.2 1"/>
-  </material>
   <!-- v2mini body -->
   <include filename="$(find v2mini_description)/urdf/v2mini_body.urdf.xacro" />

Commit message: added missing CMakeLists

File: v2mini_description/urdf/v2mini_body.urdf.xacro (robot description, xacro)
@@ -15,4 +15,10 @@
   <!-- **** BASE **** -->
   <link name="base_link">
+    <!-- fake inertial values -->
+    <inertial>
+      <mass value="1"/>
+      <inertia ixx="100" ixy="0" ixz="0" iyy="100" iyz="0" izz="100" />
+      <origin/>
+    </inertial>
     <visual>
       <origin xyz="0 0 ${base_offset_z}" rpy="0 0 0" />
@@ -35,4 +41,10 @@
   <!-- **** TORSO **** -->
   <link name="torso_link">
+    <!-- fake inertial values -->
+    <inertial>
+      <mass value="1"/>
+      <inertia ixx="100" ixy="0" ixz="0" iyy="100" iyz="0" izz="100" />
+      <origin/>
+    </inertial>
     <visual>
       <origin xyz="0 0 0" rpy="0 0 0" />
@@ -48,5 +60,5 @@
     <origin xyz="0 0 ${base_offset_z}"/>
     <axis xyz="0 0 1"/>
-    <limit effort="1000.0" lower="-0.09" upper="0" velocity="0.5"/>
+    <limit effort="10" lower="-0.09" upper="0" velocity="0.5"/>
   </joint>
 </xacro:macro>

File: v2mini_description/urdf/v2mini_robot.urdf.xacro (robot description, xacro)
@@ -38,5 +38,5 @@
     <axis xyz="0 0 1"/>
     <origin xyz="0 0 0"/>
-    <limit effort="1000.0" lower="-2.9" upper="2.9" velocity="0.1"/>
+    <limit effort="10" lower="-2.9" upper="2.9" velocity="10"/>
   </joint>
   <xacro:body/>
