Commit message: end effector change in config

File: v2mini_description/urdf/v2mini.urdf (robot description, URDF)
Before this commit: robot v2mini, 14 links, 13 joints
Joints:
- removed joint arm_joint2.0
- removed joint arm_joint3.0
- removed joint arm_joint4.0
- removed joint arm_joint5.0
- added joint arm_joint2: type revolute, parent arm_link2, child arm_link3, origin xyz=-0.026 0 0, axis 0 1 0, limit lower=-1.7 upper=1.7 effort=1000.0 velocity=0.1
- added joint arm_joint3: type revolute, parent arm_link3, child arm_link4, origin xyz=-0.0855 0 0, axis 1 0 0, limit lower=-3.1 upper=3.1 effort=1000.0 velocity=0.1
- added joint arm_joint4: type revolute, parent arm_link4, child arm_link5, origin xyz=-0.026 0 0, axis 0 0 1, limit lower=-3 upper=0.05 effort=1000.0 velocity=0.1
- added joint arm_joint5: type revolute, parent arm_link5, child arm_link6, origin xyz=0 -0.0415 0, axis 0 1 0, limit lower=-3.1 upper=3.1 effort=1000.0 velocity=0.1

File: v2mini_description/urdf/v2mini_arm.urdf.xacro (robot description, xacro)
@@ -31,11 +31,11 @@
     <limit effort="1000.0" lower="-3.1" upper="3.1" velocity="0.1"/>
   </joint>
-  <xacro:arm_link num="3" mat="black" parent="arm_link2" axis="0 1 0" offset="-0.026 0 0" roll="0" limit_low="-1.7" limit_high="1.7"/>
-  <xacro:arm_link num="4" mat="grey" parent="arm_link3" axis="1 0 0" offset="-0.0855 0 0" roll="0" limit_low="-3.1"  limit_high="3.1"/>
-  <xacro:arm_link num="5" mat="black" parent="arm_link4" axis="0 0 1" offset="-0.026 0 0" roll="${pi}" limit_low="-3" limit_high="0.05"/>
-  <xacro:arm_link num="6" mat="red" parent="arm_link5" axis="0 1 0" offset="0 -0.0415 0" roll="0" limit_low="-3.1"  limit_high="3.1"/>
+  <xacro:arm_link num="3" mat="black" par_num="2" axis="0 1 0" offset="-0.026 0 0" roll="0" limit_low="-1.7" limit_high="1.7"/>
+  <xacro:arm_link num="4" mat="grey" par_num="3" axis="1 0 0" offset="-0.0855 0 0" roll="0" limit_low="-3.1"  limit_high="3.1"/>
+  <xacro:arm_link num="5" mat="black" par_num="4" axis="0 0 1" offset="-0.026 0 0" roll="${pi}" limit_low="-3" limit_high="0.05"/>
+  <xacro:arm_link num="6" mat="red" par_num="5" axis="0 1 0" offset="0 -0.0415 0" roll="0" limit_low="-3.1"  limit_high="3.1"/>
 </xacro:macro>
 <!-- macro for the rest of the links -->
-<xacro:macro name="arm_link" params="num mat parent axis offset roll limit_low limit_high">
+<xacro:macro name="arm_link" params="num mat par_num axis offset roll limit_low limit_high">
   <link name="arm_link${num}">
     <visual>
@@ -47,6 +47,6 @@
     </visual>
   </link>
-  <joint name="arm_joint${num-1}" type="revolute">
-    <parent link="${parent}"/>
+  <joint name="arm_joint${par_num}" type="revolute">
+    <parent link="arm_link${par_num}"/>
     <child link="arm_link${num}"/>
     <origin xyz="${offset}"/>

Commit message: urdf fixed. dynamixel_jsp works

File: v2mini_description/urdf/v2mini.urdf (robot description, URDF)
Before this commit: robot v2mini, 14 links, 13 joints
Links:
- added link ee_link; collision box size=0.01 0.01 0.01
- link base_link: mass None -> 1
- link torso_link: mass None -> 1
Joints:
- added joint ee_joint: type fixed, parent arm_link6, child ee_link, origin xyz=0 0 0 rpy=0 0 0
- joint arm_joint1: origin xyz=-0.158825 -0.002 0.407507 -> xyz=-0.158825 -0.002 0.407507 rpy=3.14159 3.14159 0
- joint arm_joint2: axis 0 1 0 -> -1 0 0; origin xyz=-0.026 0 0 -> xyz=0.026 0 0 rpy=1.570795 0 4.712385
- joint arm_joint3: origin xyz=-0.0855 0 0 -> xyz= 0 0 -0.0855 rpy=0 1.570795 0
- joint arm_joint4: axis 0 0 1 -> -1 0 0; limit lower=-3 upper=0.05 effort=1000.0 velocity=0.1 -> lower=-3 upper=3 effort=1000.0 velocity=0.1; origin xyz=-0.026 0 0 -> xyz=0.026 0 0 rpy= -1.570795 0 1.570795
- joint arm_joint5: axis 0 1 0 -> -1 0 0; origin xyz=0 -0.0415 0 -> xyz=0  0 -0.0415 rpy=-1.570795 -1.570795 0
- joint body_with_head: limit lower=-2.9 upper=2.9 effort=1000.0 velocity=0.1 -> lower=-2.9 upper=2.9 effort=10 velocity=10
- joint torso_slide: limit lower=-0.09 upper=0 effort=1000.0 velocity=0.5 -> lower=-0.09 upper=0 effort=10 velocity=0.5

File: v2mini_description/urdf/v2mini_arm.urdf.xacro (robot description, xacro)
@@ -18,5 +18,5 @@
   <link name="arm_link2">
     <visual>
-      <origin xyz="0 0 0" rpy="0 0 0" />
+      <origin xyz="0 0 0" rpy="0 ${pi} 0" />
       <geometry>
         <mesh filename="package://v2mini_description/meshes/arm/arm_link2.stl" />
@@ -28,11 +28,11 @@
     <parent link="arm_link1"/>
     <child link="arm_link2"/>
-    <origin xyz="${base_offsetx} ${base_offsety} ${base_offsetz}"/>
+    <origin xyz="${base_offsetx} ${base_offsety} ${base_offsetz}" rpy="${pi} ${pi} 0"/>
     <limit effort="1000.0" lower="-3.1" upper="3.1" velocity="0.1"/>
   </joint>
-  <xacro:arm_link num="3" mat="black" par_num="2" axis="0 1 0" offset="-0.026 0 0" roll="0" limit_low="-1.7" limit_high="1.7"/>
-  <xacro:arm_link num="4" mat="grey" par_num="3" axis="1 0 0" offset="-0.0855 0 0" roll="0" limit_low="-3.1"  limit_high="3.1"/>
-  <xacro:arm_link num="5" mat="black" par_num="4" axis="0 0 1" offset="-0.026 0 0" roll="${pi}" limit_low="-3" limit_high="0.05"/>
-  <xacro:arm_link num="6" mat="red" par_num="5" axis="0 1 0" offset="0 -0.0415 0" roll="0" limit_low="-3.1"  limit_high="3.1"/>
+  <xacro:arm_link num="3" mat="black" par_num="2" axis="-1 0 0" offset="0.026 0 0" j_rpy="${pi/2} 0 ${3*pi/2}" l_rpy="0 ${-pi/2}  ${-pi/2}" limit_low="-1.7" limit_high="1.7"/>
+  <xacro:arm_link num="4" mat="grey" par_num="3" axis="1 0 0" offset=" 0 0 -0.0855" j_rpy="0 ${pi/2} 0" l_rpy="${pi/2} ${pi}  0" limit_low="-3.1"  limit_high="3.1"/>
+  <xacro:arm_link num="5" mat="black" par_num="4" axis="-1 0 0" offset="0.026 0 0" j_rpy=" ${-pi/2} 0 ${pi/2}" l_rpy="${-pi/2} 0 ${-pi/2}" limit_low="-3" limit_high="3"/>
+  <xacro:arm_link num="6" mat="red" par_num="5" axis="-1 0 0" offset="0  0 -0.0415" j_rpy="${-pi/2} ${-pi/2} 0" l_rpy="${pi/2} ${pi/2} 0" limit_low="-3.1"  limit_high="3.1"/>
   <joint name="ee_joint" type="fixed">
       <parent link="arm_link6"/>
@@ -51,8 +51,8 @@
 </xacro:macro>
 <!-- macro for the rest of the links -->
-<xacro:macro name="arm_link" params="num mat par_num axis offset roll limit_low limit_high">
+<xacro:macro name="arm_link" params="num mat par_num axis offset j_rpy l_rpy limit_low limit_high ">
   <link name="arm_link${num}">
     <visual>
-      <origin xyz="0 0 0" rpy="${roll} 0 0" />
+      <origin xyz="0 0 0" rpy="${l_rpy}" />
       <geometry>
         <mesh filename="package://v2mini_description/meshes/arm/arm_link${num}.stl" />
@@ -64,5 +64,5 @@
     <parent link="arm_link${par_num}"/>
     <child link="arm_link${num}"/>
-    <origin xyz="${offset}"/>
+    <origin xyz="${offset}" rpy="${j_rpy}"/>
     <axis xyz="${axis}"/>
     <limit effort="1000.0" lower="${limit_low}" upper="${limit_high}" velocity="0.1"/>

Commit message: added r200 to urdf

File: v2mini_description/urdf/v2mini.urdf (robot description, URDF)
Before this commit: robot v2mini, 15 links, 14 joints
Links:
- added link camera_depth_frame
- added link camera_depth_optical_frame
- added link camera_ir2_frame
- added link camera_ir2_optical_frame
- added link camera_ir_frame
- added link camera_ir_optical_frame
- added link camera_link; visual box size=0.102 0.0095 0.0038
- added link camera_rgb_frame
- added link camera_rgb_optical_frame
- link arm_link1: geometry collision mesh filename=package://v2mini_description/meshes/arm/arm_link1.stl; visual mesh filename=package://v2mini_description/meshes/arm/arm_link1.stl
- link arm_link2: geometry collision mesh filename=package://v2mini_description/meshes/arm/arm_link2.stl; visual mesh filename=package://v2mini_description/meshes/arm/arm_link2.stl
- link arm_link3: geometry collision mesh filename=package://v2mini_description/meshes/arm/arm_link3.stl; visual mesh filename=package://v2mini_description/meshes/arm/arm_link3.stl
- link arm_link4: geometry collision mesh filename=package://v2mini_description/meshes/arm/arm_link4.stl; visual mesh filename=package://v2mini_description/meshes/arm/arm_link4.stl
- link arm_link5: geometry collision mesh filename=package://v2mini_description/meshes/arm/arm_link5.stl; visual mesh filename=package://v2mini_description/meshes/arm/arm_link5.stl
- link arm_link6: geometry collision mesh filename=package://v2mini_description/meshes/arm/arm_link6.stl; visual mesh filename=package://v2mini_description/meshes/arm/arm_link6.stl
Joints:
- added joint camera_depth_joint: type fixed, parent camera_rgb_frame, child camera_depth_frame, origin xyz=0 0 0 rpy=0 0 0
- added joint camera_depth_optical_joint: type fixed, parent camera_depth_frame, child camera_depth_optical_frame, origin xyz=0 0 0 rpy=0 0 0
- added joint camera_ir2_joint: type fixed, parent camera_rgb_frame, child camera_ir2_frame, origin xyz=0 0 0 rpy=0 0 0
- added joint camera_ir2_optical_joint: type fixed, parent camera_ir2_frame, child camera_ir2_optical_frame, origin xyz=0 0 0 rpy=0 0 0
- added joint camera_ir_joint: type fixed, parent camera_rgb_frame, child camera_ir_frame, origin xyz=0 0 0 rpy=0 0 0
- added joint camera_ir_optical_joint: type fixed, parent camera_ir_frame, child camera_ir_optical_frame, origin xyz=0 0 0 rpy=0 0 0
- added joint camera_joint: type fixed, parent head_link, child camera_link, origin xyz=0 -0.0668 0.0877 rpy=0 0 0
- added joint camera_rgb_joint: type fixed, parent camera_link, child camera_rgb_frame, origin xyz=0 0 0 rpy=0 0 0
- added joint camera_rgb_optical_joint: type fixed, parent camera_rgb_frame, child camera_rgb_optical_frame, origin xyz=0 0 0 rpy=0 0 0

File: v2mini_description/urdf/v2mini_robot.urdf.xacro (robot description, xacro)
@@ -26,4 +26,6 @@
   <!-- v2mini head -->
   <include filename="$(find v2mini_description)/urdf/v2mini_head.urdf.xacro" />
+  <!-- r200 sensor -->
+  <include filename="$(find v2mini_description)/urdf/r200.urdf.xacro" />
   <!-- join the body with arm -->
   <joint name="body_with_arm" type="fixed">
@@ -43,3 +45,4 @@
   <xacro:arm/>
   <xacro:head/>
+  <xacro:sensor_r200 parent="head_link"/>
 </robot>

Commit message: constrained arm in urdf

File: v2mini_description/urdf/v2mini.urdf (robot description, URDF)
Before this commit: robot v2mini, 24 links, 23 joints
Joints:
- removed joint body_with_arm
- removed joint body_with_head
- added joint neckpan: type revolute, parent torso_link, child neck_link, origin xyz=0 0 0, axis 0 0 1, limit lower=-2.9 upper=2.9 effort=10 velocity=10
- added joint shoulder: type fixed, parent torso_link, child arm_link1, origin xyz=0 0 0

File: v2mini_description/urdf/v2mini_arm.urdf.xacro (robot description, xacro)
@@ -41,10 +41,10 @@
     <child link="arm_link2"/>
     <origin xyz="${base_offsetx} ${base_offsety} ${base_offsetz}" rpy="${pi} ${pi} 0"/>
-    <limit effort="1000.0" lower="-3.1" upper="3.1" velocity="0.1"/>
+    <limit effort="1000.0" lower="-0.2" upper="2.85" velocity="0.1"/>
   </joint>
-  <xacro:arm_link num="3" mat="black" par_num="2" axis="-1 0 0" offset="0.026 0 0" j_rpy="${pi/2} 0 ${3*pi/2}" l_rpy="0 ${-pi/2}  ${-pi/2}" limit_low="-1.7" limit_high="1.7"/>
-  <xacro:arm_link num="4" mat="grey" par_num="3" axis="1 0 0" offset=" 0 0 -0.0855" j_rpy="0 ${pi/2} 0" l_rpy="${pi/2} ${pi}  0" limit_low="-3.1"  limit_high="3.1"/>
-  <xacro:arm_link num="5" mat="black" par_num="4" axis="-1 0 0" offset="0.026 0 0" j_rpy=" ${-pi/2} 0 ${pi/2}" l_rpy="${-pi/2} 0 ${-pi/2}" limit_low="-3" limit_high="3"/>
-  <xacro:arm_link num="6" mat="red" par_num="5" axis="-1 0 0" offset="0  0 -0.0415" j_rpy="${-pi/2} ${-pi/2} 0" l_rpy="${pi/2} ${pi/2} 0" limit_low="-3.1"  limit_high="3.1"/>
+  <xacro:arm_link num="3" mat="black" par_num="2" axis="-1 0 0" offset="0.026 0 0" j_rpy="${pi/2} 0 ${3*pi/2}" l_rpy="0 ${-pi/2}  ${-pi/2}" limit_low="-0.2" limit_high="1.6"/>
+  <xacro:arm_link num="4" mat="grey" par_num="3" axis="1 0 0" offset=" 0 0 -0.0855" j_rpy="0 ${pi/2} 0" l_rpy="${pi/2} ${pi}  0" limit_low="-1.5"  limit_high="1.5"/>
+  <xacro:arm_link num="5" mat="black" par_num="4" axis="-1 0 0" offset="0.026 0 0" j_rpy=" ${-pi/2} 0 ${pi/2}" l_rpy="${-pi/2} 0 ${-pi/2}" limit_low="-1.5" limit_high="1.5"/>
+  <xacro:arm_link num="6" mat="red" par_num="5" axis="-1 0 0" offset="0  0 -0.0415" j_rpy="${-pi/2} ${-pi/2} 0" l_rpy="${pi/2} ${pi/2} 0" limit_low="-1.5"  limit_high="1.5"/>
   <joint name="ee_joint" type="fixed">
       <parent link="arm_link6"/>

File: v2mini_description/urdf/v2mini_robot.urdf.xacro (robot description, xacro)
@@ -29,5 +29,5 @@
   <include filename="$(find v2mini_description)/urdf/r200.urdf.xacro" />
   <!-- join the body with arm -->
-  <joint name="body_with_arm" type="fixed">
+  <joint name="shoulder" type="fixed">
     <parent link="torso_link"/>
     <child link="arm_link1"/>
@@ -35,5 +35,5 @@
   </joint>
   <!-- join the body with head -->
-  <joint name="body_with_head" type="revolute">
+  <joint name="neckpan" type="revolute">
     <parent link="torso_link"/>
     <child link="neck_link"/>
