Commit message: finished urdf visual

File: v2mini_description/urdf/v2mini_arm.urdf.xacro (robot description, xacro)
@@ -1,18 +1,10 @@
 <?xml version="1.0"?>
 <robot xmlns:xacro="http://www.ros.org/wiki/xacro" name="v2mini">
-  <material name="black">
-    <color rgba="0.1 0.1 0.1 1"/>
-  </material>
-  <material name="grey">
-    <color rgba="0.4 0.4 0.4 1"/>
-  </material>
-  <material name="red">
-    <color rgba="0.6 0.2 0.2 1"/>
-  </material>
-  <xacro:property name="pi" value="3.14159" />
-  <xacro:property name="base_offsetx" value="-0.158825" />
-  <xacro:property name="base_offsety" value="-0.002" />
-  <xacro:property name="base_offsetz" value="0.407507" />
-  <link name="base_link">
+<xacro:property name="pi" value="3.14159" />
+<xacro:property name="base_offsetx" value="-0.158825" />
+<xacro:property name="base_offsety" value="-0.002" />
+<xacro:property name="base_offsetz" value="0.407507" />
+<xacro:macro name="arm">
+  <link name="arm_link1">
     <visual>
       <origin xyz="0 0 0" rpy="0 0 0" />
@@ -33,30 +25,33 @@
     </visual>
   </link>
-  <joint name="arm_joint1" type="continuous">
-    <parent link="base_link"/>
+  <joint name="arm_joint1" type="revolute">
+    <parent link="arm_link1"/>
     <child link="arm_link2"/>
     <origin xyz="${base_offsetx} ${base_offsety} ${base_offsetz}"/>
+    <limit effort="1000.0" lower="-3.1" upper="3.1" velocity="0.1"/>
   </joint>
-  <!-- macro for the rest of the links -->
-  <xacro:macro name="arm_link" params="num mat parent axis offset roll">
-    <link name="arm_link${num}">
-      <visual>
-        <origin xyz="0 0 0" rpy="${roll} 0 0" />
-        <geometry>
-          <mesh filename="package://v2mini_description/meshes/arm/arm_link${num}.stl" />
-        </geometry>
-        <material name="${mat}"/>
-      </visual>
-    </link>
-    <joint name="arm_joint${num-1}" type="continuous">
-      <parent link="${parent}"/>
-      <child link="arm_link${num}"/>
-      <origin xyz="${offset}"/>
-      <axis xyz="${axis}"/>
-    </joint>
-  </xacro:macro>
-  <xacro:arm_link num="3" mat="black" parent="arm_link2" axis="0 1 0" offset="-0.026 0 0" roll="0"/>
-  <xacro:arm_link num="4" mat="grey" parent="arm_link3" axis="1 0 0" offset="-0.0855 0 0" roll="0"/>
-  <xacro:arm_link num="5" mat="black" parent="arm_link4" axis="0 0 1" offset="-0.026 0 0" roll="0"/>
-  <xacro:arm_link num="6" mat="red" parent="arm_link5" axis="0 1 0" offset="0 0.0415 0" roll="${pi}"/>
+  <xacro:arm_link num="3" mat="black" parent="arm_link2" axis="0 1 0" offset="-0.026 0 0" roll="0" limit_low="-1.7" limit_high="1.7"/>
+  <xacro:arm_link num="4" mat="grey" parent="arm_link3" axis="1 0 0" offset="-0.0855 0 0" roll="0" limit_low="-3.1"  limit_high="3.1"/>
+  <xacro:arm_link num="5" mat="black" parent="arm_link4" axis="0 0 1" offset="-0.026 0 0" roll="${pi}" limit_low="0.05" limit_high="-3"/>
+  <xacro:arm_link num="6" mat="red" parent="arm_link5" axis="0 1 0" offset="0 -0.0415 0" roll="0" limit_low="-3.1"  limit_high="3.1"/>
+</xacro:macro>
+<!-- macro for the rest of the links -->
+<xacro:macro name="arm_link" params="num mat parent axis offset roll limit_low limit_high">
+  <link name="arm_link${num}">
+    <visual>
+      <origin xyz="0 0 0" rpy="${roll} 0 0" />
+      <geometry>
+        <mesh filename="package://v2mini_description/meshes/arm/arm_link${num}.stl" />
+      </geometry>
+      <material name="${mat}"/>
+    </visual>
+  </link>
+  <joint name="arm_joint${num-1}" type="revolute">
+    <parent link="${parent}"/>
+    <child link="arm_link${num}"/>
+    <origin xyz="${offset}"/>
+    <axis xyz="${axis}"/>
+    <limit effort="1000.0" lower="${limit_low}" upper="${limit_high}" velocity="0.1"/>
+  </joint>
+</xacro:macro>
 </robot>

File: v2mini_description/urdf/v2mini_body.urdf.xacro (robot description, xacro)
@@ -1,64 +1,24 @@
 <?xml version="1.0"?>
 <robot xmlns:xacro="http://www.ros.org/wiki/xacro" name="v2mini">
-  <!-- materials -->
-  <material name="white">
-    <color rgba="0.6 0.6 0.6 1"/>
-  </material>
-  <material name="blue">
-    <color rgba="0.3 0.3 0.9 1"/>
-  </material>
-  <material name="black">
-    <color rgba="0.2 0.2 0.2 1"/>
-  </material>
-  <material name="grey">
-    <color rgba="0.4 0.4 0.4 1"/>
-  </material>
-  <material name="yellow">
-    <color rgba="0.5 0.5 0.1 1"/>
-  </material>
-  <material name="red">
-    <color rgba="0.6 0.2 0.2 1"/>
-  </material>
-  <xacro:property name="pi" value="3.14159" />
-  <!-- base properties -->
-  <xacro:property name="base_collision_height" value="0.132" />
-  <xacro:property name="base_collision_radius" value="0.175" />
-  <!-- wheel properties -->
-  <xacro:property name="wheel_radius" value="0.03" />
-  <xacro:property name="wheel_offset_radial" value="0.1405" />
-  <!-- torso properties -->
-  <xacro:property name="torso_offset_z" value="0.175" />
-  <xacro:property name="torso_width" value="0.2373" />
-  <!-- head properties -->
-  <xacro:property name="head_offset_z" value="0.2" />
-  <!-- arm properties -->
-  <xacro:property name="motor_depth" value="0.04175" />
-  <!-- materials -->
-  <material name="white">
-    <color rgba="0.6 0.6 0.6 1"/>
-  </material>
-  <material name="blue">
-    <color rgba="0.3 0.3 0.9 1"/>
-  </material>
-  <material name="black">
-    <color rgba="0.2 0.2 0.2 1"/>
-  </material>
-  <material name="grey">
-    <color rgba="0.4 0.4 0.4 1"/>
-  </material>
-  <material name="yellow">
-    <color rgba="0.5 0.5 0.1 1"/>
-  </material>
-  <material name="red">
-    <color rgba="0.6 0.2 0.2 1"/>
-  </material>
+<xacro:property name="pi" value="3.14159" />
+<!-- base properties -->
+<xacro:property name="base_offset_z" value="0.0192" />
+<xacro:property name="base_collision_height" value="0.132" />
+<xacro:property name="base_collision_radius" value="0.175" />
+<!-- wheel properties -->
+<xacro:property name="wheel_radius" value="0.03" />
+<xacro:property name="wheel_offset_radial" value="0.1405" />
+<!-- torso properties -->
+<xacro:property name="torso_offset_z" value="0.175" />
+<xacro:property name="torso_width" value="0.2373" />
+<xacro:macro name="body">
   <!-- **** BASE **** -->
   <link name="base_link">
     <visual>
-      <origin xyz="0 0 0" rpy="0 0 0" />
+      <origin xyz="0 0 ${base_offset_z}" rpy="0 0 0" />
       <geometry>
         <mesh filename="package://v2mini_description/meshes/base/base.stl" />
       </geometry>
-      <material name="yellow"/>
+      <material name="white"/>
     </visual>
     <collision>
@@ -69,22 +29,4 @@
     </collision>
   </link>
-  <!-- Macro for creating base wheels -->
-  <xacro:macro name="wheel" params="prefix reflect rotate front_set">
-    <link name="${prefix}_wheel">
-      <visual>
-        <origin xyz="0 0 0" rpy="0 0 ${pi/2*rotate}"/>
-        <geometry>
-          <mesh filename="package://v2mini_description/meshes/base/base_wheel.stl" />
-        </geometry>
-        <material name="black"/>
-      </visual>
-    </link>
-    <joint name="${prefix}_axel" type="continuous">
-      <parent link="base_link"/>
-      <child link="${prefix}_wheel"/>
-      <origin xyz="${wheel_offset_radial*reflect*(1-front_set)} ${wheel_offset_radial*reflect*front_set} 0"/>
-      <axis xyz="${1-front_set} ${front_set} 0"/>
-    </joint>
-  </xacro:macro>
   <xacro:wheel prefix="front" reflect="-1" rotate="0" front_set="1"/>
   <xacro:wheel prefix="back" reflect="1" rotate="2" front_set="1"/>
@@ -98,5 +40,5 @@
         <mesh filename="package://v2mini_description/meshes/torso/torso.stl" />
       </geometry>
-      <material name="blue"/>
+      <material name="white"/>
     </visual>
   </link>
@@ -104,7 +46,26 @@
     <parent link="base_link"/>
     <child link="torso_link"/>
-    <origin xyz="0 0 0"/>
+    <origin xyz="0 0 ${base_offset_z}"/>
     <axis xyz="0 0 1"/>
     <limit effort="1000.0" lower="-0.09" upper="0" velocity="0.5"/>
   </joint>
+</xacro:macro>
+<!-- Macro for creating base wheels -->
+<xacro:macro name="wheel" params="prefix reflect rotate front_set">
+  <link name="${prefix}_wheel">
+    <visual>
+      <origin xyz="0 0 0" rpy="0 0 ${pi/2*rotate}"/>
+      <geometry>
+        <mesh filename="package://v2mini_description/meshes/base/base_wheel.stl" />
+      </geometry>
+      <material name="red"/>
+    </visual>
+  </link>
+  <joint name="${prefix}_axel" type="continuous">
+    <parent link="base_link"/>
+    <child link="${prefix}_wheel"/>
+    <origin xyz="${wheel_offset_radial*reflect*(1-front_set)} ${wheel_offset_radial*reflect*front_set} ${wheel_radius}"/>
+    <axis xyz="${1-front_set} ${front_set} 0"/>
+  </joint>
+</xacro:macro>
 </robot>

File: v2mini_description/urdf/v2mini_robot.urdf.xacro (robot description, xacro)
@@ -1,7 +1,45 @@
 <?xml version="1.0"?>
 <robot xmlns:xacro="http://www.ros.org/wiki/xacro" name="v2mini">
+  <!-- materials -->
+  <material name="white">
+    <color rgba="0.7 0.7 0.7 1"/>
+  </material>
+  <material name="blue">
+    <color rgba="0.3 0.3 0.9 1"/>
+  </material>
+  <material name="black">
+    <color rgba="0.2 0.2 0.2 1"/>
+  </material>
+  <material name="grey">
+    <color rgba="0.4 0.4 0.4 1"/>
+  </material>
+  <material name="yellow">
+    <color rgba="0.5 0.5 0.1 1"/>
+  </material>
+  <material name="red">
+    <color rgba="0.6 0.2 0.2 1"/>
+  </material>
   <!-- v2mini body -->
   <include filename="$(find v2mini_description)/urdf/v2mini_body.urdf.xacro" />
   <!-- v2mini arm -->
   <include filename="$(find v2mini_description)/urdf/v2mini_arm.urdf.xacro" />
+  <!-- v2mini head -->
+  <include filename="$(find v2mini_description)/urdf/v2mini_head.urdf.xacro" />
+  <!-- join the body with arm -->
+  <joint name="body_with_arm" type="fixed">
+    <parent link="torso_link"/>
+    <child link="arm_link1"/>
+    <origin xyz="0 0 0"/>
+  </joint>
+  <!-- join the body with head -->
+  <joint name="body_with_head" type="revolute">
+    <parent link="torso_link"/>
+    <child link="neck_link"/>
+    <axis xyz="0 0 1"/>
+    <origin xyz="0 0 0"/>
+    <limit effort="1000.0" lower="-2.9" upper="2.9" velocity="0.1"/>
+  </joint>
+  <xacro:body/>
+  <xacro:arm/>
+  <xacro:head/>
 </robot>

Commit message: Added ee link

File: v2mini_description/urdf/v2mini_arm.urdf.xacro (robot description, xacro)
@@ -35,4 +35,18 @@
   <xacro:arm_link num="5" mat="black" par_num="4" axis="0 0 1" offset="-0.026 0 0" roll="${pi}" limit_low="-3" limit_high="0.05"/>
   <xacro:arm_link num="6" mat="red" par_num="5" axis="0 1 0" offset="0 -0.0415 0" roll="0" limit_low="-3.1"  limit_high="3.1"/>
+  <joint name="ee_joint" type="fixed">
+      <parent link="arm_link6"/>
+      <child link="ee_link"/>
+      <origin xyz="0 0 0" rpy="0 0 0"/>
+  </joint>
+  <!-- Add end effector -->
+  <link name="ee_link">
+  <collision>
+      <geometry>
+          <box size="0.01 0.01 0.01"/>
+      </geometry>
+     <origin rpy="0 0 0" xyz="0 0 0"/>
+  </collision>
+  </link>
 </xacro:macro>
 <!-- macro for the rest of the links -->

Commit message: added collision tags to arm

File: v2mini_description/urdf/v2mini_arm.urdf.xacro (robot description, xacro)
@@ -14,4 +14,10 @@
       <material name="black"/>
     </visual>
+    <collision>
+      <origin xyz="0 0 0" rpy="0 0 0"/>
+      <geometry>
+         <mesh filename="package://v2mini_description/meshes/arm_link1.stl" />
+      </geometry>
+    </collision>
   </link>
   <!-- first additional joint at offset -->
@@ -24,4 +30,10 @@
       <material name="grey"/>
     </visual>
+    <collision>
+       <origin xyz="0 0 0" rpy="0 0 0"/>
+       <geometry>
+            <mesh filename="package://v2mini_description/meshes/arm_link2.stl" />
+       </geometry>
+    </collision>
   </link>
   <joint name="arm_joint1" type="revolute">
@@ -60,4 +72,10 @@
       <material name="${mat}"/>
     </visual>
+    <collision>
+        <origin xyz="0 0 0" rpy="0 0 0"/>
+        <geometry>
+            <mesh filename="package://v2mini_description/meshes/arm/arm_link${num}.stl" />
+        </geometry>
+    </collision>
   </link>
   <joint name="arm_joint${par_num}" type="revolute">

Commit message: fixed pathingg

File: v2mini_description/urdf/v2mini_arm.urdf.xacro (robot description, xacro)
@@ -17,5 +17,5 @@
       <origin xyz="0 0 0" rpy="0 0 0"/>
       <geometry>
-         <mesh filename="package://v2mini_description/meshes/arm_link1.stl" />
+         <mesh filename="package://v2mini_description/meshes/arm/arm_link1.stl" />
       </geometry>
     </collision>
@@ -33,5 +33,5 @@
        <origin xyz="0 0 0" rpy="0 0 0"/>
        <geometry>
-            <mesh filename="package://v2mini_description/meshes/arm_link2.stl" />
+            <mesh filename="package://v2mini_description/meshes/arm/arm_link2.stl" />
        </geometry>
     </collision>

Commit message: passed in params to collision

File: v2mini_description/urdf/v2mini_arm.urdf.xacro (robot description, xacro)
@@ -31,5 +31,5 @@
     </visual>
     <collision>
-       <origin xyz="0 0 0" rpy="0 0 0"/>
+       <origin xyz="0 0 0" rpy="0 ${pi} 0"/>
        <geometry>
             <mesh filename="package://v2mini_description/meshes/arm/arm_link2.stl" />
@@ -73,5 +73,5 @@
     </visual>
     <collision>
-        <origin xyz="0 0 0" rpy="0 0 0"/>
+        <origin xyz="0 0 0" rpy="${l_rpy}"/>
         <geometry>
             <mesh filename="package://v2mini_description/meshes/arm/arm_link${num}.stl" />

Commit message: Robot spawns but masses wrng

File: v2mini_description/urdf/v2mini_arm.urdf.xacro (robot description, xacro)
@@ -20,4 +20,9 @@
       </geometry>
     </collision>
+    <inertial>
+       <origin xyz="0 0 0" rpy="0 0 0"/>
+       <mass value="1"/>
+       <inertia ixx="1.0" ixy="0.0" ixz="0.0" iyy="1.0" iyz="0.0" izz="1.0"/>
+    </inertial>
   </link>
   <!-- first additional joint at offset -->
@@ -36,4 +41,9 @@
        </geometry>
     </collision>
+   <inertial>
+       <origin xyz="0 0 0" rpy="0 0 0"/>
+       <mass value="1"/>
+       <inertia ixx="1.0" ixy="0.0" ixz="0.0" iyy="1.0" iyz="0.0" izz="1.0"/>
+    </inertial>
   </link>
   <joint name="arm_joint1" type="revolute">
@@ -60,4 +70,9 @@
      <origin rpy="0 0 0" xyz="0 0 0"/>
   </collision>
+   <inertial>
+       <origin xyz="0 0 0" rpy="0 0 0"/>
+       <mass value="1"/>
+       <inertia ixx="1.0" ixy="0.0" ixz="0.0" iyy="1.0" iyz="0.0" izz="1.0"/>
+    </inertial>
   </link>
 </xacro:macro>
@@ -78,4 +93,9 @@
         </geometry>
     </collision>
+    <inertial>
+       <origin xyz="0 0 0" rpy="0 0 0"/>
+       <mass value="1"/>
+       <inertia ixx="1.0" ixy="0.0" ixz="0.0" iyy="1.0" iyz="0.0" izz="1.0"/>
+    </inertial>
   </link>
   <joint name="arm_joint${par_num}" type="revolute">

File: v2mini_description/urdf/v2mini_head.urdf.xacro (robot description, xacro)
@@ -11,4 +11,9 @@
       <material name="black"/>
     </visual>
+     <inertial>
+       <origin xyz="0 0 0" rpy="0 0 0"/>
+       <mass value="1"/>
+       <inertia ixx="1.0" ixy="0.0" ixz="0.0" iyy="1.0" iyz="0.0" izz="1.0"/>
+    </inertial>
   </link>
   <link name="head_link">
@@ -20,4 +25,9 @@
       <material name="yellow"/>
     </visual>
+     <inertial>
+       <origin xyz="0 0 0" rpy="0 0 0"/>
+       <mass value="1"/>
+       <inertia ixx="1.0" ixy="0.0" ixz="0.0" iyy="1.0" iyz="0.0" izz="1.0"/>
+    </inertial>
   </link>
   <joint name="neck_tilt" type="revolute">

File: v2mini_gazebo/urdf/transmission/v2mini_arm.transmission.xacro (robot description, xacro)
@@ -2,10 +2,10 @@
 <robot xmlns:xacro="http://ros.org/wiki/xacro">
   <xacro:macro name="v2mini_arm_transmission" params="prefix">
-    <transmission name="${prefix}arm_joint1_trans">
+ <transmission name="${prefix}arm_joint2_trans">
       <type>transmission_interface/SimpleTransmission</type>
-      <joint name="${prefix}arm_joint1">
+      <joint name="${prefix}arm_joint2">
         <hardwareInterface>PositionJointInterface</hardwareInterface>
       </joint>
-      <actuator name="${prefix}arm_joint1_motor">
+      <actuator name="${prefix}arm_joint2_motor">
         <mechanicalReduction>1</mechanicalReduction>
       </actuator>
@@ -47,13 +47,4 @@
       </actuator>
     </transmission>
-   <transmission name="${prefix}arm_joint6_trans">
-      <type>transmission_interface/SimpleTransmission</type>
-      <joint name="${prefix}arm_joint6">
-        <hardwareInterface>PositionJointInterface</hardwareInterface>
-      </joint>
-      <actuator name="${prefix}arm_joint6_motor">
-        <mechanicalReduction>1</mechanicalReduction>
-      </actuator>
-    </transmission>
   </xacro:macro>
 </robot>

File: v2mini_gazebo/urdf/v2mini_robot.gazebo.xacro (robot description, xacro)
@@ -1,6 +1,6 @@
 <?xml version="1.0"?>
-<robot xmlns:xacro="http://ros.org/wiki/xacro">
+<robot xmlns:xacro="http://ros.org/wiki/xacro" name="v2mini">
   <!-- Includes -->
-  <xacro:include filename="$(find v2mini_description)/urdf/gazebo/transmission/v2mini_arm.transmission.xacro"/>
+  <xacro:include filename="$(find v2mini_gazebo)/urdf/transmission/v2mini_arm.transmission.xacro"/>
   <xacro:include filename="$(find v2mini_description)/urdf/v2mini_robot.urdf.xacro"/>
   <!-- Add the gazebo plugins here -->

Commit message: upd

File: v2mini_description/urdf/v2mini_arm.urdf.xacro (robot description, xacro)
@@ -22,5 +22,5 @@
     <inertial>
        <origin xyz="0 0 0" rpy="0 0 0"/>
-       <mass value="1"/>
+       <mass value="0.01"/>
        <inertia ixx="1.0" ixy="0.0" ixz="0.0" iyy="1.0" iyz="0.0" izz="1.0"/>
     </inertial>
@@ -43,5 +43,5 @@
    <inertial>
        <origin xyz="0 0 0" rpy="0 0 0"/>
-       <mass value="1"/>
+       <mass value="0.01"/>
        <inertia ixx="1.0" ixy="0.0" ixz="0.0" iyy="1.0" iyz="0.0" izz="1.0"/>
     </inertial>
@@ -95,5 +95,5 @@
     <inertial>
        <origin xyz="0 0 0" rpy="0 0 0"/>
-       <mass value="1"/>
+       <mass value="0.01"/>
        <inertia ixx="1.0" ixy="0.0" ixz="0.0" iyy="1.0" iyz="0.0" izz="1.0"/>
     </inertial>

File: v2mini_description/urdf/v2mini_body.urdf.xacro (robot description, xacro)
@@ -17,5 +17,5 @@
     <!-- fake inertial values -->
     <inertial>
-      <mass value="1"/>
+      <mass value="10"/>
       <inertia ixx="100" ixy="0" ixz="0" iyy="100" iyz="0" izz="100" />
       <origin/>
@@ -43,5 +43,5 @@
     <!-- fake inertial values -->
     <inertial>
-      <mass value="1"/>
+      <mass value="5"/>
       <inertia ixx="100" ixy="0" ixz="0" iyy="100" iyz="0" izz="100" />
       <origin/>
@@ -73,4 +73,9 @@
       <material name="red"/>
     </visual>
+     <inertial>
+       <origin xyz="0 0 0" rpy="0 0 0"/>
+       <mass value="1"/>
+       <inertia ixx="1.0" ixy="0.0" ixz="0.0" iyy="1.0" iyz="0.0" izz="1.0"/>
+    </inertial>
   </link>
   <joint name="${prefix}_axel" type="continuous">
