Commit message: Added joint1

File: v2mini_gazebo/urdf/transmission/v2mini_arm.transmission.xacro (robot description, xacro)
@@ -2,10 +2,10 @@
 <robot xmlns:xacro="http://ros.org/wiki/xacro">
   <xacro:macro name="v2mini_arm_transmission" params="prefix">
- <transmission name="${prefix}arm_joint2_trans">
+   <transmission name="${prefix}arm_joint1_trans">
       <type>transmission_interface/SimpleTransmission</type>
-      <joint name="${prefix}arm_joint2">
+      <joint name="${prefix}arm_joint1">
         <hardwareInterface>PositionJointInterface</hardwareInterface>
       </joint>
-      <actuator name="${prefix}arm_joint2_motor">
+      <actuator name="${prefix}arm_joint1_motor">
         <mechanicalReduction>1</mechanicalReduction>
       </actuator>
